Commit message: Rename joints

File: packages/lemodel/so101_description/urdf/so101_macro.xacro (robot description, xacro)
@@ -330,5 +330,5 @@
     </joint>
     <!-- Joint from wrist to gripper -->
-    <joint name="wrist_roll" type="revolute">
+    <joint name="joint_5" type="revolute">
       <origin xyz="5.55112e-17 -0.0611 0.0181" rpy="1.5708 0.0486795 3.14159"/>
       <parent link="${prefix}wrist_link"/>
@@ -338,5 +338,5 @@
     </joint>
     <!-- Joint from lower_arm to wrist -->
-    <joint name="wrist_flex" type="revolute">
+    <joint name="joint_4" type="revolute">
       <origin xyz="-0.1349 0.0052 3.62355e-17" rpy="4.02456e-15 8.67362e-16 -1.5708"/>
       <parent link="${prefix}lower_arm_link"/>
@@ -347,5 +347,5 @@
     <!-- Joint from upper_arm to lower_arm -->
     <!-- Note: 5-degree calibration offset applied to joint limits -->
-    <joint name="elbow_flex" type="revolute">
+    <joint name="joint_3" type="revolute">
       <origin xyz="-0.11257 -0.028 1.73763e-16" rpy="-3.63608e-16 8.74301e-16 1.5708"/>
       <parent link="${prefix}upper_arm_link"/>
@@ -355,5 +355,5 @@
     </joint>
     <!-- Joint from shoulder to upper_arm -->
-    <joint name="shoulder_lift" type="revolute">
+    <joint name="joint_2" type="revolute">
       <origin xyz="-0.0303992 -0.0182778 -0.0542" rpy="-1.5708 -1.5708 0"/>
       <parent link="${prefix}shoulder_link"/>
@@ -363,5 +363,5 @@
     </joint>
     <!-- Joint from base to shoulder -->
-    <joint name="shoulder_pan" type="revolute">
+    <joint name="joint_1" type="revolute">
       <origin xyz="0.0388353 -8.97657e-09 0.0624" rpy="3.14159 4.18253e-17 -3.14159"/>
       <parent link="${prefix}base_link"/>

File: packages/lemodel/so101_description/urdf/so101_ros2_control.xacro (robot description, xacro)
@@ -10,5 +10,5 @@
         <param name="calibration_file">${calibration_file}</param>
       </hardware>
-      <joint name="shoulder_pan">
+      <joint name="joint_1">
         <command_interface name="position">
           <param name="min">-1.91986</param>
@@ -19,5 +19,5 @@
         <state_interface name="current"/>
       </joint>
-      <joint name="shoulder_lift">
+      <joint name="joint_2">
         <command_interface name="position">
           <param name="min">-1.74533</param>
@@ -28,5 +28,5 @@
         <state_interface name="current"/>
       </joint>
-      <joint name="elbow_flex">
+      <joint name="joint_3">
         <command_interface name="position">
           <param name="min">-1.69</param>
@@ -37,5 +37,5 @@
         <state_interface name="current"/>
       </joint>
-      <joint name="wrist_flex">
+      <joint name="joint_4">
         <command_interface name="position">
           <param name="min">-1.65806</param>
@@ -46,5 +46,5 @@
         <state_interface name="current"/>
       </joint>
-      <joint name="wrist_roll">
+      <joint name="joint_5">
         <command_interface name="position">
           <param name="min">-2.74385</param>

Commit message: Rename links

File: packages/lemodel/so101_description/urdf/so101_macro.xacro (robot description, xacro)
@@ -12,6 +12,12 @@
       <color rgba="0.1 0.1 0.1 1.0"/>
     </material>
+    <link name="${prefix}base_link"></link>
+    <joint name="${prefix}base_joint" type="fixed">
+      <parent link="${prefix}base_link"/>
+      <child link="${prefix}link_1"/>
+      <origin xyz="0 0 0" rpy="0 0 0"/>
+    </joint>
     <!-- Link base -->
-    <link name="${prefix}base_link">
+    <link name="${prefix}link_1">
       <inertial>
         <origin xyz="0.0137179 -5.19711e-05 0.0334843" rpy="0 0 0"/>
@@ -77,5 +83,5 @@
     </link>
     <!-- Link shoulder -->
-    <link name="${prefix}shoulder_link">
+    <link name="${prefix}link_2">
       <inertial>
         <origin xyz="-0.0307604 -1.66727e-05 -0.0252713" rpy="0 0 0"/>
@@ -127,5 +133,5 @@
     </link>
     <!-- Link upper_arm -->
-    <link name="${prefix}upper_arm_link">
+    <link name="${prefix}link_3">
       <inertial>
         <origin xyz="-0.0898471 -0.00838224 0.0184089" rpy="0 0 0"/>
@@ -163,5 +169,5 @@
     </link>
     <!-- Link lower_arm -->
-    <link name="${prefix}lower_arm_link">
+    <link name="${prefix}link_4">
       <inertial>
         <origin xyz="-0.0980701 0.00324376 0.0182831" rpy="0 0 0"/>
@@ -213,5 +219,5 @@
     </link>
     <!-- Link wrist -->
-    <link name="${prefix}wrist_link">
+    <link name="${prefix}link_5">
       <inertial>
         <origin xyz="-0.000103312 -0.0386143 0.0281156" rpy="0 0 0"/>
@@ -332,5 +338,5 @@
     <joint name="joint_5" type="revolute">
       <origin xyz="5.55112e-17 -0.0611 0.0181" rpy="1.5708 0.0486795 3.14159"/>
-      <parent link="${prefix}wrist_link"/>
+      <parent link="${prefix}link_5"/>
       <child link="${prefix}gripper_link"/>
       <axis xyz="0 0 1"/>
@@ -340,6 +346,6 @@
     <joint name="joint_4" type="revolute">
       <origin xyz="-0.1349 0.0052 3.62355e-17" rpy="4.02456e-15 8.67362e-16 -1.5708"/>
-      <parent link="${prefix}lower_arm_link"/>
-      <child link="${prefix}wrist_link"/>
+      <parent link="${prefix}link_4"/>
+      <child link="${prefix}link_5"/>
       <axis xyz="0 0 1"/>
       <limit effort="10" velocity="10" lower="-1.65806" upper="1.65806"/>
@@ -349,6 +355,6 @@
     <joint name="joint_3" type="revolute">
       <origin xyz="-0.11257 -0.028 1.73763e-16" rpy="-3.63608e-16 8.74301e-16 1.5708"/>
-      <parent link="${prefix}upper_arm_link"/>
-      <child link="${prefix}lower_arm_link"/>
+      <parent link="${prefix}link_3"/>
+      <child link="${prefix}link_4"/>
       <axis xyz="0 0 1"/>
       <limit effort="10" velocity="10" lower="-1.69" upper="1.69"/>
@@ -357,6 +363,6 @@
     <joint name="joint_2" type="revolute">
       <origin xyz="-0.0303992 -0.0182778 -0.0542" rpy="-1.5708 -1.5708 0"/>
-      <parent link="${prefix}shoulder_link"/>
-      <child link="${prefix}upper_arm_link"/>
+      <parent link="${prefix}link_2"/>
+      <child link="${prefix}link_3"/>
       <axis xyz="0 0 1"/>
       <limit effort="10" velocity="10" lower="-1.74533" upper="1.74533"/>
@@ -365,6 +371,6 @@
     <joint name="joint_1" type="revolute">
       <origin xyz="0.0388353 -8.97657e-09 0.0624" rpy="3.14159 4.18253e-17 -3.14159"/>
-      <parent link="${prefix}base_link"/>
-      <child link="${prefix}shoulder_link"/>
+      <parent link="${prefix}link_1"/>
+      <child link="${prefix}link_2"/>
       <axis xyz="0 0 1"/>
       <limit effort="10" velocity="10" lower="-1.91986" upper="1.91986"/>
